Commit message: working nbv

File: yak_ur5_support/urdf/yak_ur5_workcell.urdf.xacro (robot description, xacro)
@@ -4,5 +4,5 @@
 <!-- |    EDITING THIS FILE BY HAND IS NOT RECOMMENDED                                 | -->
 <!-- =================================================================================== -->
-<robot name="yak_ur3_workcell" xmlns:xacro="http://ros.org/wiki/xacro">
+<robot name="yak_ur5_workcell" xmlns:xacro="http://ros.org/wiki/xacro">
   <!-- measured from model -->
   <!--property name="shoulder_height" value="0.089159" /-->
@@ -294,4 +294,5 @@
   </joint>
   <link name="world_frame"/>
+  <link name="tsdf_frame"/>
   <link name="stand">
     <origin rpy="0 0 0" xyz="0 0 0"/>
@@ -307,4 +308,36 @@
       <geometry>
         <cylinder length="1.0414" radius="0.0762"/>
+      </geometry>
+    </collision>
+  </link>
+  <link name="right_wall">
+    <origin rpy="0 0 0" xyz="0 0 0"/>
+    <visual>
+      <geometry>
+        <box size="2 .1 2"/>
+      </geometry>
+      <material name="blue">
+        <color rgba="1 1 1 1"/>
+      </material>
+    </visual>
+    <collision>
+      <geometry>
+        <box size="2 .1 2"/>
+      </geometry>
+    </collision>
+  </link>
+  <link name="back_wall">
+    <origin rpy="0 0 0" xyz="0 0 0"/>
+    <visual>
+      <geometry>
+        <box size=".1 2 2"/>
+      </geometry>
+      <material name="blue">
+        <color rgba="1 1 1 1"/>
+      </material>
+    </visual>
+    <collision>
+      <geometry>
+        <box size=".1 2 2"/>
       </geometry>
     </collision>
@@ -347,3 +380,19 @@
     <origin rpy="-1.57 0.0 0.0" xyz="0.0 0.0 0.0"/>
   </joint>
+  <!-- todo these paremeters need to  be synced with kinfu node loanch params -->
+  <joint name="world_frame_to_tsdf_frame" type="fixed">
+    <parent link="world_frame"/>
+    <child link="tsdf_frame"/>
+    <origin rpy="0.0 0.0 0.0" xyz="0.4 -0.5 1"/>
+  </joint>
+  <joint name="world_to_right_wall" type="fixed">
+    <parent link="world_frame"/>
+    <child link="right_wall"/>
+    <origin rpy="0.0 0.0 0.0" xyz="0 -0.8636 1"/>
+  </joint>
+  <joint name="world_to_back_wall" type="fixed">
+    <parent link="world_frame"/>
+    <child link="back_wall"/>
+    <origin rpy="0.0 0.0 0.0" xyz="-1 0.0 1"/>
+  </joint>
 </robot>

File: yak_ur5_support/urdf/yak_ur5_workcell.xacro (robot description, xacro)
@@ -1,4 +1,4 @@
 <?xml version="1.0" ?>
-<robot name="yak_ur3_workcell" xmlns:xacro="http://ros.org/wiki/xacro">
+<robot name="yak_ur5_workcell" xmlns:xacro="http://ros.org/wiki/xacro">
   <xacro:include filename="$(find ur_description)/urdf/ur5.urdf.xacro"/>
   <xacro:ur5_robot prefix="" joint_limited="true"/>
@@ -7,4 +7,5 @@
   <xacro:property name="inch_to_meter" value="0.0254" />
   <link name="world_frame"/>
+  <link name="tsdf_frame"/>
   <link name="stand">
     <origin xyz="0 0 0" rpy="0 0 0" />
@@ -20,4 +21,36 @@
       <geometry>
         <cylinder length="${41*inch_to_meter}" radius="${3*inch_to_meter}" />
+      </geometry>
+    </collision>
+  </link>
+  <link name="right_wall">
+    <origin xyz="0 0 0" rpy="0 0 0" />
+    <visual>
+      <geometry>
+        <box size="2 .1 2" />
+      </geometry>
+      <material name="blue">
+          <color rgba="1 1 1 1"/>
+      </material>
+    </visual>
+    <collision>
+      <geometry>
+        <box size="2 .1 2" />
+      </geometry>
+    </collision>
+  </link>
+  <link name="back_wall">
+    <origin xyz="0 0 0" rpy="0 0 0" />
+    <visual>
+      <geometry>
+        <box size=".1 2 2" />
+      </geometry>
+      <material name="blue">
+          <color rgba="1 1 1 1"/>
+      </material>
+    </visual>
+    <collision>
+      <geometry>
+        <box size=".1 2 2" />
       </geometry>
     </collision>
@@ -60,3 +93,19 @@
     <origin xyz="0.0 0.0 0.0" rpy="-1.57 0.0 0.0" />
   </joint>
+  <!-- todo these paremeters need to  be synced with kinfu node loanch params -->
+  <joint name="world_frame_to_tsdf_frame" type="fixed">
+    <parent link="world_frame" />
+    <child link = "tsdf_frame" />
+    <origin xyz="0.4 -0.5 1" rpy="0.0 0.0 0.0" />
+  </joint>
+  <joint name="world_to_right_wall" type="fixed">
+    <parent link="world_frame" />
+    <child link = "right_wall" />
+    <origin xyz="0 -0.8636 1" rpy="0.0 0.0 0.0" />
+  </joint>
+  <joint name="world_to_back_wall" type="fixed">
+    <parent link="world_frame" />
+    <child link = "back_wall" />
+    <origin xyz="-1 0.0 1" rpy="0.0 0.0 0.0" />
+  </joint>
 </robot>
